Commit message: [CleanTheTableDemo] fixed some issues

File: resources/robocup_clean_v1.urdf (robot description, URDF)
Before this commit: robot iai-kitchen, 110 links, 109 joints
Links:
- removed link coathanger:coathanger:coathanger_center
- removed link coathanger:coathanger:coathanger_front_edge_center
- removed link coathanger:coathanger:coathanger_origin
- removed link dishwasher_table:d_table:d_table_origin
- removed link lamp:lamp:lamp_center
- removed link lamp:lamp:lamp_front_edge_center
- removed link lamp:lamp:lamp_origin
- removed link suturo_couch:couch:place_one
- removed link suturo_couch:couch:place_three
- removed link suturo_couch:couch:place_two
- removed link trashcan:trashcan:trashcan_center
- removed link trashcan:trashcan:trashcan_front_edge_center
- removed link trashcan:trashcan:trashcan_origin
- removed link wall_1_link
- removed link wall_2_link
- removed link wall_3_link
- removed link wall_4_link
- removed link wall_5_link
- removed link wall_6_link
- removed link wall_7_link
- removed link wall_8_link
- added link coathanger:coathanger:table_center, mass 1.0; collision box size=0.5 0.5 1.8; visual box size=0.5 0.5 1.8
- added link coathanger:coathanger:table_front_edge_center
- added link coathanger:coathanger:table_origin
- added link dishwasher_table:d_table:table_origin
- added link suturo_couch:couch:place1
- added link suturo_couch:couch:place2, mass 1.0; collision box size=0.65 0.725 0.3; visual box size=0.65 0.725 0.3
- added link suturo_couch:couch:place3, mass 1.0; collision box size=0.65 0.725 0.3; visual box size=0.65 0.725 0.3
- added link trashcan:trashcan:table_center, mass 1.0; collision cylinder length=0.49 radius=0.19; visual cylinder length=0.49 radius=0.19
- added link trashcan:trashcan:table_front_edge_center
- added link trashcan:trashcan:table_origin
Joints:
- removed joint coathanger:coathanger:coathanger_front_edge_center_joint
- removed joint coathanger:coathanger:coathanger_origin_joint
- removed joint lamp:lamp:center_joint
- removed joint lamp:lamp:lamp_front_edge_center_joint
- removed joint lamp:lamp:lamp_origin_joint
- removed joint trashcan:trashcan:trashcan_front_edge_center_joint
- removed joint trashcan:trashcan:trashcan_origin_joint
- removed joint wall_1_center_joint
- removed joint wall_2_center_joint
- removed joint wall_3_center_joint
- removed joint wall_4_center_joint
- removed joint wall_5_center_joint
- removed joint wall_6_center_joint
- removed joint wall_7_center_joint
- removed joint wall_8_center_joint
- added joint coathanger:coathanger:table_front_edge_center_joint: type fixed, parent coathanger:coathanger:table_origin, child coathanger:coathanger:table_front_edge_center, origin xyz=0.0 0.25 1.8 rpy=0.0 0.0 0.0
- added joint coathanger:coathanger:table_origin_joint: type fixed, parent urdf_offset, child coathanger:coathanger:table_origin, origin xyz=3.9 1.55 0.0 rpy=0.0 0.0 3.17
- added joint trashcan:trashcan:table_front_edge_center_joint: type fixed, parent trashcan:trashcan:table_origin, child trashcan:trashcan:table_front_edge_center, origin xyz=0.0 0.0 0.49 rpy=0.0 0.0 0.0
- added joint trashcan:trashcan:table_origin_joint: type fixed, parent urdf_offset, child trashcan:trashcan:table_origin, origin xyz=5.86 2.03 0.0 rpy=0.0 0.0 3.2
- joint coathanger:coathanger:center_joint: child coathanger:coathanger:coathanger_center -> coathanger:coathanger:table_center; parent coathanger:coathanger:coathanger_origin -> coathanger:coathanger:table_origin
- joint dish_washer_table_center_joint: parent dishwasher_table:d_table:d_table_origin -> dishwasher_table:d_table:table_origin
- joint dish_washer_table_edge_joint: parent dishwasher_table:d_table:d_table_origin -> dishwasher_table:d_table:table_origin
- joint dish_washer_table_main_joint: child dishwasher_table:d_table:d_table_origin -> dishwasher_table:d_table:table_origin
- joint iai_kitchen:arena:door_handle_inside_joint: origin xyz=-0.069 0.0 0.06 rpy=0.0 0.0 1.5707963267948966 -> xyz=-0.0635 0.0 0.06 rpy=0.0 0.0 1.5707963267948966
- joint office:arena:door_handle_inside_joint: origin xyz=-0.069 0.0 0.06 rpy=0.0 0.0 1.5707963267948966 -> xyz=-0.0635 0.0 0.06 rpy=0.0 0.0 1.5707963267948966
- joint suturo_couch:couch:couch_left_joint: child suturo_couch:couch:place_two -> suturo_couch:couch:place2; parent suturo_couch:couch:place_one -> suturo_couch:couch:place1
- joint suturo_couch:couch:couch_origin_joint: child suturo_couch:couch:place_one -> suturo_couch:couch:place1
- joint suturo_couch:couch:couch_right_joint: child suturo_couch:couch:place_three -> suturo_couch:couch:place3; parent suturo_couch:couch:place_one -> suturo_couch:couch:place1
- joint trashcan:trashcan:center_joint: child trashcan:trashcan:trashcan_center -> trashcan:trashcan:table_center; parent trashcan:trashcan:trashcan_origin -> trashcan:trashcan:table_origin
