Commit message: [gripper_tool_frame] adjusted name of tool frame to "hand_gripper_tool_frame"

File: resources/robots/hsrb.urdf (robot description, URDF)
Before this commit: robot hsrb, 46 links, 45 joints
Links:
- removed link gripper_tool_frame
- added link hand_gripper_tool_frame
Joints:
- removed joint gripper_tool_joint
- added joint hand_gripper_tool_joint: type fixed, parent wrist_roll_link, child hand_gripper_tool_frame, origin xyz=0.0 0.0 0.23090002 rpy=0.0 0.0 1.5707963267948963
